File: KiCad-8 Files/DSS-SSR4E.kicad_pcb (KiCad board)
At the start: 2 copper layers, 49 x 54.1 mm, 46 parts, among them J1 IDC 26 HDR, J2 Phoenix_1844811, Q1 BSL606SN, Q2 BSL606SN, Q3 BSL606SN, Q4 BSL606SN, U1 CD74ACT540, U2 IL613E

Commit message: update kicad files for OSHWA cert.
Parts:
- added G***: LOGO, Custom_Footprints:OSHWA_US002623, F.Cu at (205.1, 125.1)
